Commit message: .

File: src/fairino_description/urdf/fairino5_v6.urdf (robot description, URDF)
Before this commit: robot fairino5_v6_robot, 7 links, 6 joints
Links:
- added link ee_link; visual cylinder length=0.05 radius=0.003; visual cylinder length=0.05 radius=0.003
Joints:
- added joint wrist3_to_ee: type fixed, parent wrist3_link, child ee_link, origin xyz=0 0 0.1 rpy=0 0 0

Commit message: .broken

File: src/fairino_description/urdf/fairino5_v6.urdf (robot description, URDF)
Before this commit: robot fairino5_v6_robot, 8 links, 7 joints
Links:
- link ee_link: mass None -> 0.1; geometry collision mesh filename=package://fairino_description/meshes/disk.stl scale=0.001 0.001 0.001; visual cylinder length=0.05 radius=0.003

Commit message: .broken

File: src/fairino_description/urdf/fairino5_v6.urdf (robot description, URDF)
Before this commit: robot fairino5_v6_robot, 9 links, 8 joints
Links:
- added link mounting_surface; collision mesh filename=package://fairino_description/meshes/Cobot - Plot.stl; visual mesh filename=package://fairino_description/meshes/Cobot - Plot.stl
Joints:
- added joint world_to_mount: type fixed, parent world, child mounting_surface, origin xyz=0 0 0 rpy=0 0 0

Commit message: FIX SUB MM MOVES

File: src/fairino_description/urdf/fairino5_v6.urdf (robot description, URDF)
Before this commit: robot fairino5_v6_robot, 10 links, 9 joints
Links:
- link ee_link: geometry collision mesh filename=package://fairino_description/meshes/disk.stl scale=0.001 0.001 0.001; visual cylinder length=0.05 radius=0.003

Commit message: FIX SUB MM MOVES

File: src/fairino_description/urdf/fairino5_v6.urdf (robot description, URDF)
Before this commit: robot fairino5_v6_robot, 10 links, 9 joints
Links:
- link mounting_surface: geometry collision box size=0.4764 0.1417 0.3579; collision box size=0.9048 1.2167 0.0250
