Commit message: Add drag mode functionality and collision monitoring support for eRobo3 robot

File: eRob_moveit/src/eRob_ROS2_MoveIt/zeroerr/config/eRobo3.ros2_control.xacro (robot description, xacro)
@@ -9,8 +9,15 @@
                 <param name="master_id">0</param>
                 <param name="control_frequency">1000</param>
+                <param name="freeze_on_slave_fault">true</param>
                 <param name="timeout">1000000000</param>
             </hardware>
             <joint name="Joint_1">
                 <command_interface name="position">
+                </command_interface>
+                <command_interface name="mode_of_operation">
+                </command_interface>
+                <command_interface name="effort">
+                </command_interface>
+                <command_interface name="torque_offset">
                 </command_interface>
                 <command_interface name="reset_fault"/>
@@ -20,4 +27,9 @@
                 <state_interface name="velocity"/>
                 <state_interface name="effort"/>
+                <state_interface name="motor_actual_current"/>
+                <state_interface name="following_error_actual"/>
+                <state_interface name="statusword"/>
+                <state_interface name="error_code"/>
+                <state_interface name="mode_display"/>
                 <ec_module name="zero_err1">
 		  <plugin>ethercat_generic_plugins/EcCiA402Drive</plugin>
@@ -31,4 +43,10 @@
                 <command_interface name="position">
                 </command_interface>
+                <command_interface name="mode_of_operation">
+                </command_interface>
+                <command_interface name="effort">
+                </command_interface>
+                <command_interface name="torque_offset">
+                </command_interface>
                 <command_interface name="reset_fault"/>
                 <command_interface name="enable_set"/>
@@ -37,4 +55,9 @@
                 <state_interface name="velocity"/>
                 <state_interface name="effort"/>
+                <state_interface name="motor_actual_current"/>
+                <state_interface name="following_error_actual"/>
+                <state_interface name="statusword"/>
+                <state_interface name="error_code"/>
+                <state_interface name="mode_display"/>
                 <ec_module name="zero_err2">
 		  <plugin>ethercat_generic_plugins/EcCiA402Drive</plugin>
@@ -48,4 +71,10 @@
                 <command_interface name="position">
                 </command_interface>
+                <command_interface name="mode_of_operation">
+                </command_interface>
+                <command_interface name="effort">
+                </command_interface>
+                <command_interface name="torque_offset">
+                </command_interface>
                 <command_interface name="reset_fault"/>
                 <command_interface name="enable_set"/>
@@ -54,4 +83,9 @@
                 <state_interface name="velocity"/>
                 <state_interface name="effort"/>
+                <state_interface name="motor_actual_current"/>
+                <state_interface name="following_error_actual"/>
+                <state_interface name="statusword"/>
+                <state_interface name="error_code"/>
+                <state_interface name="mode_display"/>
                 <ec_module name="zero_err3">
 		  <plugin>ethercat_generic_plugins/EcCiA402Drive</plugin>
@@ -65,4 +99,10 @@
                 <command_interface name="position">
                 </command_interface>
+                <command_interface name="mode_of_operation">
+                </command_interface>
+                <command_interface name="effort">
+                </command_interface>
+                <command_interface name="torque_offset">
+                </command_interface>
                 <command_interface name="reset_fault"/>
                 <command_interface name="enable_set"/>
@@ -71,4 +111,9 @@
                 <state_interface name="velocity"/>
                 <state_interface name="effort"/>
+                <state_interface name="motor_actual_current"/>
+                <state_interface name="following_error_actual"/>
+                <state_interface name="statusword"/>
+                <state_interface name="error_code"/>
+                <state_interface name="mode_display"/>
                 <ec_module name="zero_err4">
 		  <plugin>ethercat_generic_plugins/EcCiA402Drive</plugin>
@@ -82,4 +127,10 @@
                 <command_interface name="position">
                 </command_interface>
+                <command_interface name="mode_of_operation">
+                </command_interface>
+                <command_interface name="effort">
+                </command_interface>
+                <command_interface name="torque_offset">
+                </command_interface>
                 <command_interface name="reset_fault"/>
                 <command_interface name="enable_set"/>
@@ -88,4 +139,9 @@
                 <state_interface name="velocity"/>
                 <state_interface name="effort"/>
+                <state_interface name="motor_actual_current"/>
+                <state_interface name="following_error_actual"/>
+                <state_interface name="statusword"/>
+                <state_interface name="error_code"/>
+                <state_interface name="mode_display"/>
                 <ec_module name="zero_err5">
 		  <plugin>ethercat_generic_plugins/EcCiA402Drive</plugin>
@@ -99,4 +155,10 @@
                 <command_interface name="position">
                 </command_interface>
+                <command_interface name="mode_of_operation">
+                </command_interface>
+                <command_interface name="effort">
+                </command_interface>
+                <command_interface name="torque_offset">
+                </command_interface>
                 <command_interface name="reset_fault"/>
                 <command_interface name="enable_set"/>
@@ -105,4 +167,9 @@
                 <state_interface name="velocity"/>
                 <state_interface name="effort"/>
+                <state_interface name="motor_actual_current"/>
+                <state_interface name="following_error_actual"/>
+                <state_interface name="statusword"/>
+                <state_interface name="error_code"/>
+                <state_interface name="mode_display"/>
                 <ec_module name="zero_err6">
 		  <plugin>ethercat_generic_plugins/EcCiA402Drive</plugin>

File: eRob_moveit/src/eRob_ROS2_MoveIt/zeroerr/config/erob_arm.urdf (robot description, URDF)
Before this commit: robot eRobo3, 11 links, 10 joints
Links:
- link Link_2: geometry collision mesh filename=package://zeroerr/meshes/Link_2.stl scale=1.00000 1.00000 1.00000; visual mesh filename=package://zeroerr/meshes/Link_2.stl scale=1.00000 1.00000 1.00000
- link Link_3: geometry collision mesh filename=package://zeroerr/meshes/Link_3.stl scale=1.00000 1.00000 1.00000; visual mesh filename=package://zeroerr/meshes/Link_3.stl scale=1.00000 1.00000 1.00000
Joints:
- joint Joint_3: origin xyz=0.00000 0.00050 0.36350 rpy=0.00000 0.00000 0.00000 -> xyz=0.00000 0.00050 0.24350 rpy=0.00000 0.00000 0.00000
- joint Joint_4: origin xyz=0.00000 -0.01400 0.31100 rpy=0.00000 0.00000 0.00000 -> xyz=0.00000 -0.01400 0.21100 rpy=0.00000 0.00000 0.00000
