Commit message: Add fairino oscilloscope script and update collision monitoring configuration
- Introduced `fairino_oscilloscope.py` for enhanced motion visualization.
- Updated `fairino_launch.conf` to include oscilloscope launch option.
- Enhanced collision monitor configuration with static torque bias and warmup parameters.
- Adjusted trajectory optimizer integration in various modules for improved motion planning.

File: eRob_moveit/src/eRob_ROS2_MoveIt/zeroerr/config/erob_arm.urdf (robot description, URDF)
Before this commit: robot eRobo3, 11 links, 10 joints
Links:
- added link ring_raster_m5; collision mesh filename=package://zeroerr/meshes/ring_raster_m5_10_centered.stl scale=0.001 0.001 0.001; visual mesh filename=package://zeroerr/meshes/ring_raster_m5_10_centered.stl scale=0.001 0.001 0.001
Joints:
- added joint ring_raster_m5_joint: type fixed, parent tool0, child ring_raster_m5, origin xyz=0 0.010 0 rpy=0 0 0
- joint tcp_joint: origin xyz=0 -0.0305 -0.083 rpy=0 0 0 -> xyz=0 0 0 rpy=0 0 0; parent tool0 -> ring_raster_m5
- joint tool0: origin xyz=0.0 0.042 -0.030 rpy=-1.5708 0.0 3.14159 -> xyz=0 0.042 0 rpy=0 0 0

File: eRob_moveit/src/eRob_ROS2_MoveIt/zeroerr/config/erob_arm_backup_corrected_mass.urdf (robot description, URDF)
Before this commit: robot eRobo3, 11 links, 10 joints
Links:
- added link ring_raster_m5; collision mesh filename=package://zeroerr/meshes/ring_raster_m5_10_centered.stl scale=0.001 0.001 0.001; visual mesh filename=package://zeroerr/meshes/ring_raster_m5_10_centered.stl scale=0.001 0.001 0.001
Joints:
- added joint ring_raster_m5_joint: type fixed, parent tool0, child ring_raster_m5, origin xyz=0 0.010 0 rpy=0 0 0
- joint tcp_joint: origin xyz=0 -0.0305 -0.083 rpy=0 0 0 -> xyz=0 0 0 rpy=0 0 0; parent tool0 -> ring_raster_m5
- joint tool0: origin xyz=0.0 0.042 -0.030 rpy=-1.5708 0.0 3.14159 -> xyz=0 0 0 rpy=0 0 0

File: eRob_moveit/src/eRob_ROS2_MoveIt/zeroerr/config/erob_arm_family_motor_masses.urdf (robot description, URDF)
Before this commit: robot eRobo3, 11 links, 10 joints
Links:
- added link ring_raster_m5; collision mesh filename=package://zeroerr/meshes/ring_raster_m5_10_centered.stl scale=0.001 0.001 0.001; visual mesh filename=package://zeroerr/meshes/ring_raster_m5_10_centered.stl scale=0.001 0.001 0.001
Joints:
- added joint ring_raster_m5_joint: type fixed, parent tool0, child ring_raster_m5, origin xyz=0 0.010 0 rpy=0 0 0
- joint tcp_joint: origin xyz=0 -0.0305 -0.083 rpy=0 0 0 -> xyz=0 0 0 rpy=0 0 0; parent tool0 -> ring_raster_m5
- joint tool0: origin xyz=0.0 0.042 -0.030 rpy=-1.5708 0.0 3.14159 -> xyz=0 0 0 rpy=0 0 0

File: src/fairino_description/urdf/fairino5_v6.urdf (robot description, URDF)
Before this commit: robot fairino5_v6_robot, 10 links, 9 joints
Links:
- added link disk_link; collision mesh filename=package://fairino_description/meshes/disk.stl scale=0.001 0.001 0.001; visual mesh filename=package://fairino_description/meshes/disk.stl scale=0.001 0.001 0.001
- link ee_link: geometry visual cylinder length=0.05 radius=0.003; visual cylinder length=0.05 radius=0.003
Joints:
- added joint ee_to_disk: type fixed, parent ee_link, child disk_link, origin xyz=0 0 0 rpy=0 0 0

Commit message: Refactor end effector naming and update collision parameters in URDF and configuration files

File: eRob_moveit/src/eRob_ROS2_MoveIt/zeroerr/config/erob_arm.urdf (robot description, URDF)
Before this commit: robot eRobo3, 12 links, 11 joints
Links:
- removed link ring_raster_m5
- removed link tcp
- removed link tool0
- added link disk_link; collision mesh filename=package://zeroerr/meshes/disk.stl scale=0.001 0.001 0.001; visual mesh filename=package://zeroerr/meshes/disk.stl scale=0.001 0.001 0.001
- added link disk_mount
- added link ee_link
Joints:
- removed joint ring_raster_m5_joint
- removed joint tcp_joint
- removed joint tool0
- added joint disk_mount_to_disk: type fixed, parent disk_mount, child disk_link, origin xyz=0 0 0 rpy=0 0 0
- added joint ee_to_disk_mount: type fixed, parent ee_link, child disk_mount, origin xyz=0 0 0 rpy=0 0 -1.1344640138
- added joint link6_to_ee: type fixed, parent Link_6, child ee_link, origin xyz=0 0 0 rpy=-1.5708 0 0

File: eRob_moveit/src/eRob_ROS2_MoveIt/zeroerr/config/erob_arm_backup_corrected_mass.urdf (robot description, URDF)
Before this commit: robot eRobo3, 12 links, 11 joints
Links:
- link ring_raster_m5: mass None -> 2.5; geometry collision mesh filename=package://zeroerr/meshes/disk.stl scale=0.001 0.001 0.001; visual mesh filename=package://zeroerr/meshes/disk.stl scale=0.001 0.001 0.001
Joints:
- joint ring_raster_m5_joint: origin xyz=0 0.010 0 rpy=0 0 0 -> xyz=0 0 0 rpy=0 0 0
- joint tcp_joint: origin xyz=0 0 0 rpy=0 0 0 -> xyz=0 0 0.1 rpy=0 0 0; parent ring_raster_m5 -> tool0
- joint tool0: origin xyz=0 0 0 rpy=0 0 0 -> xyz=0 0 0 rpy=-1.5708 0 0

File: eRob_moveit/src/eRob_ROS2_MoveIt/zeroerr/config/erob_arm_family_motor_masses.urdf (robot description, URDF)
Before this commit: robot eRobo3, 12 links, 11 joints
Links:
- removed link ring_raster_m5
- removed link tcp
- removed link tool0
- added link disk_link, mass 2.5; collision mesh filename=package://zeroerr/meshes/disk.stl scale=0.001 0.001 0.001; visual mesh filename=package://zeroerr/meshes/disk.stl scale=0.001 0.001 0.001
- added link disk_mount
- added link ee_link
Joints:
- removed joint ring_raster_m5_joint
- removed joint tcp_joint
- removed joint tool0
- added joint disk_mount_to_disk: type fixed, parent disk_mount, child disk_link, origin xyz=0 0 0 rpy=0 0 0
- added joint ee_to_disk_mount: type fixed, parent ee_link, child disk_mount, origin xyz=0 0 0 rpy=0 0 -1.1344640138
- added joint link6_to_ee: type fixed, parent Link_6, child ee_link, origin xyz=0 0 0 rpy=-1.5708 0 0

Commit message: Refactor end effector naming and update collision parameters in URDF and configuration files

File: eRob_moveit/src/eRob_ROS2_MoveIt/zeroerr/config/erob_arm.urdf (robot description, URDF)
Before this commit: robot eRobo3, 12 links, 11 joints
Links:
- link table: geometry collision box size=2.0 2.0 0.03; visual box size=2.0 2.0 0.03

File: eRob_moveit/src/eRob_ROS2_MoveIt/zeroerr/config/erob_arm_backup_corrected_mass.urdf (robot description, URDF)
Before this commit: robot eRobo3, 12 links, 11 joints
Links:
- link table: geometry collision box size=2.0 2.0 0.03; visual box size=2.0 2.0 0.03

File: eRob_moveit/src/eRob_ROS2_MoveIt/zeroerr/config/erob_arm_family_motor_masses.urdf (robot description, URDF)
Before this commit: robot eRobo3, 12 links, 11 joints
Links:
- link table: geometry collision box size=2.0 2.0 0.03; visual box size=2.0 2.0 0.03
Joints:
- joint Joint_3: limit lower=-3.14159 upper=3.14159 effort=2.0 velocity=1000.0 -> lower=-2.6 upper=0.1 effort=2.0 velocity=1000.0
- joint ee_to_disk_mount: origin xyz=0 0 0 rpy=0 0 -1.1344640138 -> xyz=0 0 0 rpy=0 0 -1.439897
