Commit message: Add fairino oscilloscope script and update collision monitoring configuration
- Introduced `fairino_oscilloscope.py` for enhanced motion visualization.
- Updated `fairino_launch.conf` to include oscilloscope launch option.
- Enhanced collision monitor configuration with static torque bias and warmup parameters.
- Adjusted trajectory optimizer integration in various modules for improved motion planning.

File: eRob_moveit/src/eRob_ROS2_MoveIt/zeroerr/config/eRobo3.urdf.xacro (robot description, xacro)
@@ -2,6 +2,7 @@
 <robot xmlns:xacro="http://www.ros.org/wiki/xacro" name="eRobo3">
     <xacro:arg name="initial_positions_file" default="initial_positions.yaml" />
-    <!-- Import eRobo3 urdf file -->
-    <xacro:include filename="$(find zeroerr)/config/erob_arm_backup_corrected_mass.urdf" />
+    <!-- Import eRobo3 urdf file — path driven by URDF_PATH in runtime.yaml via launch arg -->
+    <xacro:arg name="robot_urdf" default="$(find zeroerr)/config/erob_arm_family_motor_masses.urdf"/>
+    <xacro:include filename="$(arg robot_urdf)" />
     <!-- Import control_xacro -->
     <xacro:include filename="eRobo3.ros2_control.xacro" />

File: eRob_moveit/src/eRob_ROS2_MoveIt/zeroerr/config/erob_arm_family_motor_masses.urdf (robot description, URDF)
Before this commit: robot eRobo3, 11 links, 10 joints
Links:
- link Link_1: mass 0.50622 -> 2.44622
- link Link_2: mass 1.59000 -> 3.53000
- link Link_3: mass 1.04000 -> 2.98000
- link Link_4: mass 0.31668 -> 1.55668
- link Link_5: mass 0.31668 -> 1.55668
- link Link_6: mass 0.10121 -> 1.34121

Commit message: Update planning pipelines and adjust timing parameters in launch and configuration files

File: eRob_moveit/src/eRob_ROS2_MoveIt/zeroerr/config/eRobo3.urdf.xacro (robot description, xacro)
@@ -2,6 +2,6 @@
 <robot xmlns:xacro="http://www.ros.org/wiki/xacro" name="eRobo3">
     <xacro:arg name="initial_positions_file" default="initial_positions.yaml" />
-    <!-- Import eRobo3 urdf file — path driven by URDF_PATH in runtime.yaml via launch arg -->
-    <xacro:arg name="robot_urdf" default="$(find zeroerr)/config/erob_arm_family_motor_masses.urdf"/>
+    <!-- Import eRobo3 urdf file - launch sets ZEROERR_ROBOT_URDF from runtime.yaml. -->
+    <xacro:arg name="robot_urdf" default="$(optenv ZEROERR_ROBOT_URDF /__runtime_yaml_must_set_robot_urdf__.urdf)"/>
     <xacro:include filename="$(arg robot_urdf)" />
     <!-- Import control_xacro -->

File: eRob_moveit/src/eRob_ROS2_MoveIt/zeroerr/config/erob_arm.urdf (robot description, URDF)
Before this commit: robot eRobo3, 12 links, 11 joints
Links:
- link Link_1: geometry collision mesh filename=package://zeroerr/meshes/welding/Link_1.stl scale=1.00000 1.00000 1.00000; visual mesh filename=package://zeroerr/meshes/welding/Link_1.stl scale=1.00000 1.00000 1.00000
- link Link_2: geometry collision mesh filename=package://zeroerr/meshes/welding/Link_2.stl scale=1.00000 1.00000 1.00000; visual mesh filename=package://zeroerr/meshes/welding/Link_2.stl scale=1.00000 1.00000 1.00000
- link Link_3: geometry collision mesh filename=package://zeroerr/meshes/welding/Link_3.stl scale=1.00000 1.00000 1.00000; visual mesh filename=package://zeroerr/meshes/welding/Link_3.stl scale=1.00000 1.00000 1.00000
- link Link_4: geometry collision mesh filename=package://zeroerr/meshes/welding/Link_4.stl scale=1.00000 1.00000 1.00000; visual mesh filename=package://zeroerr/meshes/welding/Link_4.stl scale=1.00000 1.00000 1.00000
- link Link_5: geometry collision mesh filename=package://zeroerr/meshes/welding/Link_5.stl scale=1.00000 1.00000 1.00000; visual mesh filename=package://zeroerr/meshes/welding/Link_5.stl scale=1.00000 1.00000 1.00000
- link Link_6: geometry collision mesh filename=package://zeroerr/meshes/welding/Link_6.stl scale=1.00000 1.00000 1.00000; visual mesh filename=package://zeroerr/meshes/welding/Link_6.stl scale=1.00000 1.00000 1.00000
- link base_link_inertial: geometry collision mesh filename=package://zeroerr/meshes/welding/base_link.stl scale=1.00000 1.00000 1.00000; visual mesh filename=package://zeroerr/meshes/welding/base_link.stl scale=1.00000 1.00000 1.00000
- link disk_link: geometry collision mesh filename=package://zeroerr/meshes/welding/disk.stl scale=0.001 0.001 0.001; visual mesh filename=package://zeroerr/meshes/welding/disk.stl scale=0.001 0.001 0.001

File: eRob_moveit/src/eRob_ROS2_MoveIt/zeroerr/config/erob_arm_backup_corrected_mass.urdf (robot description, URDF)
Before this commit: robot eRobo3, 12 links, 11 joints
Links:
- link Link_1: geometry collision mesh filename=package://zeroerr/meshes/welding/Link_1.stl scale=1.00000 1.00000 1.00000; visual mesh filename=package://zeroerr/meshes/welding/Link_1.stl scale=1.00000 1.00000 1.00000
- link Link_2: geometry collision mesh filename=package://zeroerr/meshes/welding/Link_2_extended.stl scale=1.00000 1.00000 1.00000; visual mesh filename=package://zeroerr/meshes/welding/Link_2_extended.stl scale=1.00000 1.00000 1.00000
- link Link_3: geometry collision mesh filename=package://zeroerr/meshes/welding/Link_3_extended.stl scale=1.00000 1.00000 1.00000; visual mesh filename=package://zeroerr/meshes/welding/Link_3_extended.stl scale=1.00000 1.00000 1.00000
- link Link_4: geometry collision mesh filename=package://zeroerr/meshes/welding/Link_4.stl scale=1.00000 1.00000 1.00000; visual mesh filename=package://zeroerr/meshes/welding/Link_4.stl scale=1.00000 1.00000 1.00000
- link Link_5: geometry collision mesh filename=package://zeroerr/meshes/welding/Link_5.stl scale=1.00000 1.00000 1.00000; visual mesh filename=package://zeroerr/meshes/welding/Link_5.stl scale=1.00000 1.00000 1.00000
- link Link_6: geometry collision mesh filename=package://zeroerr/meshes/welding/Link_6.stl scale=1.00000 1.00000 1.00000; visual mesh filename=package://zeroerr/meshes/welding/Link_6.stl scale=1.00000 1.00000 1.00000
- link base_link_inertial: geometry collision mesh filename=package://zeroerr/meshes/welding/base_link.stl scale=1.00000 1.00000 1.00000; visual mesh filename=package://zeroerr/meshes/welding/base_link.stl scale=1.00000 1.00000 1.00000
- link ring_raster_m5: geometry collision mesh filename=package://zeroerr/meshes/welding/disk.stl scale=0.001 0.001 0.001; visual mesh filename=package://zeroerr/meshes/welding/disk.stl scale=0.001 0.001 0.001
