Commit message: Update planning pipelines and adjust timing parameters in launch and configuration files

File: eRob_moveit/src/eRob_ROS2_MoveIt/zeroerr/config/paint/erob_arm_small.urdf (robot description, URDF)
Before this commit: robot eRobo3, 13 links, 12 joints
Links:
- link Link_2: geometry collision mesh filename=package://zeroerr/meshes/paint/Link_2_extended.stl scale=1.00000 1.00000 1.00000; visual mesh filename=package://zeroerr/meshes/paint/Link_2_extended.stl scale=1.00000 1.00000 1.00000
- link Link_3: geometry collision mesh filename=package://zeroerr/meshes/paint/Link_3_extended.stl scale=1.00000 1.00000 1.00000; visual mesh filename=package://zeroerr/meshes/paint/Link_3_extended.stl scale=1.00000 1.00000 1.00000
Joints:
- joint Joint_3: origin xyz=0.00000 0.00050 0.24350 rpy=0.00000 0.00000 0.00000 -> xyz=0.00000 0.00050 0.36350 rpy=0.00000 0.00000 0.00000
- joint Joint_4: origin xyz=0.00000 -0.01400 0.21100 rpy=0.00000 0.00000 0.00000 -> xyz=0.00000 -0.01400 0.31100 rpy=0.00000 0.00000 0.00000
