Commit message: Refactor eRob ros2_control joints into reusable Xacro macro

File: eRob_moveit/src/eRob_ROS2_MoveIt/zeroerr/config/urdfs/eRobo3.ros2_control.xacro (robot description, xacro)
@@ -1,6 +1,13 @@
 <?xml version="1.0"?>
 <robot xmlns:xacro="http://www.ros.org/wiki/xacro">
-    <xacro:macro name="eRobo3_ros2_control" params="name initial_positions_file use_fake_hardware:=false">
-        <xacro:property name="initial_positions" value="${xacro.load_yaml(initial_positions_file)['initial_positions']}"/>
+    <!-- Reusable ros2_control joint macro -->
+    <xacro:include filename="eRob.ros2_control.macros.xacro"/>
+    <xacro:macro
+        name="eRobo3_ros2_control"
+        params="name initial_positions_file use_fake_hardware:=false">
+        <xacro:property
+            name="initial_positions"
+            value="${xacro.load_yaml(initial_positions_file)['initial_positions']}"
+        />
         <ros2_control name="${name}" type="system">
             <hardware>
@@ -16,136 +23,58 @@
                 </xacro:unless>
             </hardware>
-            <joint name="Joint_1">
-                <command_interface name="position"/>
-                <state_interface name="position">
-                    <param name="initial_value">${initial_positions['Joint_1']}</param>
-                </state_interface>
-                <state_interface name="velocity"/>
-                <state_interface name="effort"/>
-                <xacro:unless value="${use_fake_hardware}">
-                    <command_interface name="reset_fault"/>
-                    <command_interface name="enable_set"/>
-                    <command_interface name="disable_set"/>
-                    <state_interface name="statusword"/>
-                    <state_interface name="error_code"/>
-                    <state_interface name="mode_display"/>
-                    <ec_module name="zero_err1">
-                        <plugin>ethercat_generic_plugins/EcCiA402Drive</plugin>
-                        <param name="alias">0</param>
-                        <param name="position">0</param>
-                        <param name="slave_config">$(find zeroerr)/config/zeroErr.yaml</param>
-                    </ec_module>
-                </xacro:unless>
-            </joint>
-            <joint name="Joint_2">
-                <command_interface name="position"/>
-                <state_interface name="position">
-                    <param name="initial_value">${initial_positions['Joint_2']}</param>
-                </state_interface>
-                <state_interface name="velocity"/>
-                <state_interface name="effort"/>
-                <xacro:unless value="${use_fake_hardware}">
-                    <command_interface name="reset_fault"/>
-                    <command_interface name="enable_set"/>
-                    <command_interface name="disable_set"/>
-                    <state_interface name="statusword"/>
-                    <state_interface name="error_code"/>
-                    <state_interface name="mode_display"/>
-                    <ec_module name="zero_err2">
-                        <plugin>ethercat_generic_plugins/EcCiA402Drive</plugin>
-                        <param name="alias">0</param>
-                        <param name="position">1</param>
-                        <param name="slave_config">$(find zeroerr)/config/zeroErr1.yaml</param>
-                    </ec_module>
-                </xacro:unless>
-            </joint>
-            <joint name="Joint_3">
-                <command_interface name="position"/>
-                <state_interface name="position">
-                    <param name="initial_value">${initial_positions['Joint_3']}</param>
-                </state_interface>
-                <state_interface name="velocity"/>
-                <state_interface name="effort"/>
-                <xacro:unless value="${use_fake_hardware}">
-                    <command_interface name="reset_fault"/>
-                    <command_interface name="enable_set"/>
-                    <command_interface name="disable_set"/>
-                    <state_interface name="statusword"/>
-                    <state_interface name="error_code"/>
-                    <state_interface name="mode_display"/>
-                    <ec_module name="zero_err3">
-                        <plugin>ethercat_generic_plugins/EcCiA402Drive</plugin>
-                        <param name="alias">0</param>
-                        <param name="position">2</param>
-                        <param name="slave_config">$(find zeroerr)/config/zeroErr.yaml</param>
-                    </ec_module>
-                </xacro:unless>
-            </joint>
-            <joint name="Joint_4">
-                <command_interface name="position"/>
-                <state_interface name="position">
-                    <param name="initial_value">${initial_positions['Joint_4']}</param>
-                </state_interface>
-                <state_interface name="velocity"/>
-                <state_interface name="effort"/>
-                <xacro:unless value="${use_fake_hardware}">
-                    <command_interface name="reset_fault"/>
-                    <command_interface name="enable_set"/>
-                    <command_interface name="disable_set"/>
-                    <state_interface name="statusword"/>
-                    <state_interface name="error_code"/>
-                    <state_interface name="mode_display"/>
-                    <ec_module name="zero_err4">
-                        <plugin>ethercat_generic_plugins/EcCiA402Drive</plugin>
-                        <param name="alias">0</param>
-                        <param name="position">3</param>
-                        <param name="slave_config">$(find zeroerr)/config/zeroErr1.yaml</param>
-                    </ec_module>
-                </xacro:unless>
-            </joint>
-            <joint name="Joint_5">
-                <command_interface name="position"/>
-                <state_interface name="position">
-                    <param name="initial_value">${initial_positions['Joint_5']}</param>
-                </state_interface>
-                <state_interface name="velocity"/>
-                <state_interface name="effort"/>
-                <xacro:unless value="${use_fake_hardware}">
-                    <command_interface name="reset_fault"/>
-                    <command_interface name="enable_set"/>
-                    <command_interface name="disable_set"/>
-                    <state_interface name="statusword"/>
-                    <state_interface name="error_code"/>
-                    <state_interface name="mode_display"/>
-                    <ec_module name="zero_err5">
-                        <plugin>ethercat_generic_plugins/EcCiA402Drive</plugin>
-                        <param name="alias">0</param>
-                        <param name="position">4</param>
-                        <param name="slave_config">$(find zeroerr)/config/zeroErr.yaml</param>
-                    </ec_module>
-                </xacro:unless>
-            </joint>
-            <joint name="Joint_6">
-                <command_interface name="position"/>
-                <state_interface name="position">
-                    <param name="initial_value">${initial_positions['Joint_6']}</param>
-                </state_interface>
-                <state_interface name="velocity"/>
-                <state_interface name="effort"/>
-                <xacro:unless value="${use_fake_hardware}">
-                    <command_interface name="reset_fault"/>
-                    <command_interface name="enable_set"/>
-                    <command_interface name="disable_set"/>
-                    <state_interface name="statusword"/>
-                    <state_interface name="error_code"/>
-                    <state_interface name="mode_display"/>
-                    <ec_module name="zero_err6">
-                        <plugin>ethercat_generic_plugins/EcCiA402Drive</plugin>
-                        <param name="alias">0</param>
-                        <param name="position">5</param>
-                        <param name="slave_config">$(find zeroerr)/config/zeroErr.yaml</param>
-                    </ec_module>
-                </xacro:unless>
-            </joint>
+            <!-- Joint 1 -->
+            <xacro:erob_control_joint
+                joint_name="Joint_1"
+                module_name="zero_err1"
+                slave_position="0"
+                slave_config="$(find zeroerr)/config/zeroErr.yaml"
+                initial_position="${initial_positions['Joint_1']}"
+                use_fake_hardware="${use_fake_hardware}"
+            />
+            <!-- Joint 2 -->
+            <xacro:erob_control_joint
+                joint_name="Joint_2"
+                module_name="zero_err2"
+                slave_position="1"
+                slave_config="$(find zeroerr)/config/zeroErr1.yaml"
+                initial_position="${initial_positions['Joint_2']}"
+                use_fake_hardware="${use_fake_hardware}"
+            />
+            <!-- Joint 3 -->
+            <xacro:erob_control_joint
+                joint_name="Joint_3"
+                module_name="zero_err3"
+                slave_position="2"
+                slave_config="$(find zeroerr)/config/zeroErr.yaml"
+                initial_position="${initial_positions['Joint_3']}"
+                use_fake_hardware="${use_fake_hardware}"
+            />
+            <!-- Joint 4 -->
+            <xacro:erob_control_joint
+                joint_name="Joint_4"
+                module_name="zero_err4"
+                slave_position="3"
+                slave_config="$(find zeroerr)/config/zeroErr1.yaml"
+                initial_position="${initial_positions['Joint_4']}"
+                use_fake_hardware="${use_fake_hardware}"
+            />
+            <!-- Joint 5 -->
+            <xacro:erob_control_joint
+                joint_name="Joint_5"
+                module_name="zero_err5"
+                slave_position="4"
+                slave_config="$(find zeroerr)/config/zeroErr.yaml"
+                initial_position="${initial_positions['Joint_5']}"
+                use_fake_hardware="${use_fake_hardware}"
+            />
+            <!-- Joint 6 -->
+            <xacro:erob_control_joint
+                joint_name="Joint_6"
+                module_name="zero_err6"
+                slave_position="5"
+                slave_config="$(find zeroerr)/config/zeroErr.yaml"
+                initial_position="${initial_positions['Joint_6']}"
+                use_fake_hardware="${use_fake_hardware}"
+            />
         </ros2_control>
     </xacro:macro>
