Commit message: .

File: eRob_moveit/src/eRob_ROS2_MoveIt/zeroerr/config/twin_robots/urdfs/twin_erob.urdf.xacro (robot description, xacro)
@@ -11,5 +11,5 @@
   <!-- Robot 1                                                     -->
   <!-- ============================================================ -->
-  <xacro:erob_arm prefix="robot1_"/>
+  <xacro:erob_arm prefix="robot1_" use_short_links="true"/>
   <joint name="world_to_robot1_base" type="fixed">
     <parent link="world"/>
@@ -26,5 +26,5 @@
   <!-- Robot 2                                                     -->
   <!-- ============================================================ -->
-  <xacro:erob_arm prefix="robot2_"/>
+  <xacro:erob_arm prefix="robot2_" use_short_links="true"/>
   <joint name="world_to_robot2_base" type="fixed">
     <parent link="world"/>

File: eRob_moveit/src/eRob_ROS2_MoveIt/zeroerr/config/urdfs/erob_arm_macro.xacro (robot description, xacro)
@@ -11,5 +11,5 @@
       must be defined by the wrapper URDF/Xacro.
   -->
-  <xacro:macro name="erob_arm" params="prefix">
+  <xacro:macro name="erob_arm" params="prefix use_short_links:=false">
     <!-- ============================================================ -->
     <!-- Materials                                                    -->
@@ -69,7 +69,14 @@
     </joint>
     <joint name="${prefix}Joint_3" type="revolute">
-      <origin
-        rpy="0.00000 0.00000 0.00000"
-        xyz="0.00000 0.00050 0.36350"/>
+      <xacro:if value="${use_short_links}">
+        <origin
+          rpy="0.00000 0.00000 0.00000"
+          xyz="0.00000 0.00050 0.24350"/>
+      </xacro:if>
+      <xacro:unless value="${use_short_links}">
+        <origin
+          rpy="0.00000 0.00000 0.00000"
+          xyz="0.00000 0.00050 0.36350"/>
+      </xacro:unless>
       <parent link="${prefix}Link_2"/>
       <child link="${prefix}Link_3"/>
@@ -88,7 +95,14 @@
     </joint>
     <joint name="${prefix}Joint_4" type="revolute">
-      <origin
-        rpy="0.00000 0.00000 0.00000"
-        xyz="0.00000 -0.01400 0.31100"/>
+      <xacro:if value="${use_short_links}">
+        <origin
+          rpy="0.00000 0.00000 0.00000"
+          xyz="0.00000 -0.01400 0.21100"/>
+      </xacro:if>
+      <xacro:unless value="${use_short_links}">
+        <origin
+          rpy="0.00000 0.00000 0.00000"
+          xyz="0.00000 -0.01400 0.31100"/>
+      </xacro:unless>
       <parent link="${prefix}Link_3"/>
       <child link="${prefix}Link_4"/>
@@ -192,7 +206,14 @@
           xyz="0.00000 0.00000 0.00000"/>
         <geometry>
-          <mesh
-            filename="package://zeroerr/meshes/paint/Link_2_extended.stl"
-            scale="1.00000 1.00000 1.00000"/>
+          <xacro:if value="${use_short_links}">
+            <mesh
+              filename="package://zeroerr/meshes/paint/Link_2_short.stl"
+              scale="1.00000 1.00000 1.00000"/>
+          </xacro:if>
+          <xacro:unless value="${use_short_links}">
+            <mesh
+              filename="package://zeroerr/meshes/paint/Link_2_extended.stl"
+              scale="1.00000 1.00000 1.00000"/>
+          </xacro:unless>
         </geometry>
       </collision>
@@ -216,7 +237,14 @@
         <material name="${prefix}arm_material"/>
         <geometry>
-          <mesh
-            filename="package://zeroerr/meshes/paint/Link_2_extended.stl"
-            scale="1.00000 1.00000 1.00000"/>
+          <xacro:if value="${use_short_links}">
+            <mesh
+              filename="package://zeroerr/meshes/paint/Link_2_short.stl"
+              scale="1.00000 1.00000 1.00000"/>
+          </xacro:if>
+          <xacro:unless value="${use_short_links}">
+            <mesh
+              filename="package://zeroerr/meshes/paint/Link_2_extended.stl"
+              scale="1.00000 1.00000 1.00000"/>
+          </xacro:unless>
         </geometry>
       </visual>
@@ -231,7 +259,14 @@
           xyz="0.00000 0.00000 0.00000"/>
         <geometry>
-          <mesh
-            filename="package://zeroerr/meshes/paint/Link_3_extended.stl"
-            scale="1.00000 1.00000 1.00000"/>
+          <xacro:if value="${use_short_links}">
+            <mesh
+              filename="package://zeroerr/meshes/paint/Link_3_short.stl"
+              scale="1.00000 1.00000 1.00000"/>
+          </xacro:if>
+          <xacro:unless value="${use_short_links}">
+            <mesh
+              filename="package://zeroerr/meshes/paint/Link_3_extended.stl"
+              scale="1.00000 1.00000 1.00000"/>
+          </xacro:unless>
         </geometry>
       </collision>
@@ -255,7 +290,14 @@
         <material name="${prefix}arm_material"/>
         <geometry>
-          <mesh
-            filename="package://zeroerr/meshes/paint/Link_3_extended.stl"
-            scale="1.00000 1.00000 1.00000"/>
+          <xacro:if value="${use_short_links}">
+            <mesh
+              filename="package://zeroerr/meshes/paint/Link_3_short.stl"
+              scale="1.00000 1.00000 1.00000"/>
+          </xacro:if>
+          <xacro:unless value="${use_short_links}">
+            <mesh
+              filename="package://zeroerr/meshes/paint/Link_3_extended.stl"
+              scale="1.00000 1.00000 1.00000"/>
+          </xacro:unless>
         </geometry>
       </visual>
