Commit message: implented servo jog

File: eRob_moveit/src/eRob_ROS2_MoveIt/zeroerr/config/paint/urdfs/erob_arm_small.with_mounting_stl.urdf (robot description, URDF)
Before this commit: robot eRobo3, 12 links, 11 joints
Links:
- link mounting_surface: geometry collision box size=0.115 0.190 0.1475; visual mesh filename=package://zeroerr/meshes/paint/latest_mounting.stl scale=0.001 0.001 0.001
Joints:
- joint mounting_surface_joint: origin xyz=0 0 0 rpy=0 0 0 -> xyz=0 0 0 rpy=0 0 1.57079633

Commit message: adjusted mounting surface and disk stl

File: eRob_moveit/src/eRob_ROS2_MoveIt/zeroerr/config/paint/urdfs/erob_arm_small.with_mounting_stl.urdf (robot description, URDF)
Before this commit: robot eRobo3, 12 links, 11 joints
Links:
- link tool0: geometry collision mesh filename=package://zeroerr/meshes/paint/00035513_disk_origin_centere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 scale=0.001 0.001 0.001; visual mesh filename=package://zeroerr/meshes/paint/00035513_disk_origin_centere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 scale=0.001 0.001 0.001
Joints:
- joint mounting_surface_joint: origin xyz=0 0 0 rpy=0 0 1.57079633 -> xyz=-0.015219 0.015023 0.000000 rpy=0.000000 0.000000 2.856873

Commit message: The active URDF rendered the full mounting STL, but MoveIt collision geometry contained only a small fixture box. I changed the collision geometry to use latest_mounting.stl, so:
  - Solid plate regions are now collision-protected.
  - The central opening remains open.
  - Servo can detect the actual mounting surface shape.

  Verification passed:

  - URDF parsed successfully with check_urdf.
  - zeroerr built successfully.
  - The installed URDF contains the corrected mesh collision.

File: eRob_moveit/src/eRob_ROS2_MoveIt/zeroerr/config/paint/urdfs/erob_arm_small.with_mounting_stl.urdf (robot description, URDF)
Before this commit: robot eRobo3, 12 links, 11 joints
Links:
- link mounting_surface: geometry collision mesh filename=package://zeroerr/meshes/paint/latest_mounting.stl scale=0.001 0.001 0.001; visual mesh filename=package://zeroerr/meshes/paint/latest_mounting.stl scale=0.001 0.001 0.001

Commit message: Added collision geometry for the raised fixture:
  - Main housing box
  - Horizontal upper bracket
  - 300 mm vertical post cylinder
  - Wider top-cap cylinder

File: eRob_moveit/src/eRob_ROS2_MoveIt/zeroerr/config/paint/urdfs/erob_arm_small.with_mounting_stl.urdf (robot description, URDF)
Before this commit: robot eRobo3, 12 links, 11 joints
Links:
- link mounting_surface: geometry collision box size=0.007 0.207 0.008; collision box size=0.007 0.532 0.008
