Commit message: optimised dropoff return for tray_dry system

File: eRob_moveit/src/eRob_ROS2_MoveIt/zeroerr/config/paint_short_links/urdfs/erob_arm_short_links.with_mounting_stl.urdf (robot description, URDF)
Before this commit: robot eRobo3, 12 links, 11 joints
Links:
- link tcp: geometry visual sphere radius=0.00050
- link tool0: geometry collision mesh filename=package://zeroerr/meshes/paint/ToolPointer.stl scale=0.001 0.001 0.001; visual mesh filename=package://zeroerr/meshes/paint/ToolPointer.stl scale=0.001 0.001 0.001
Joints:
- joint Joint_1: limit lower=-6.28318 upper=6.28318 effort=20.0 velocity=1000.0 -> lower=-6.28318 upper=6.28318 effort=20.0 velocity=3.0; origin xyz=0.00000 0.00000 0.00000 rpy=0.00000 0.00000 1.041994390 -> xyz=0.00000 0.00000 0.00000 rpy=0.00000 0.00000 0.00000
- joint Joint_2: limit lower=-3.14159 upper=3.14159 effort=20.0 velocity=1000.0 -> lower=-3.14159 upper=3.14159 effort=20.0 velocity=3.0; origin xyz=0.00000 0.05300 0.14050 rpy=0.00000 0.035892822 0.00000 -> xyz=0.00000 0.05300 0.14050 rpy=0.00000 0.00000 0.00000
- joint Joint_3: limit lower=-3.14159 upper=3.14159 effort=20.0 velocity=1000.0 -> lower=-3.14159 upper=3.14159 effort=20.0 velocity=3.0; origin xyz=0.00000 0.00050 0.24350 rpy=0.00000 -0.036551956 0.00000 -> xyz=0.00000 0.00050 0.24350 rpy=0.00000 0.00000 0.00000
- joint Joint_4: limit lower=-4.88692 upper=3.14159 effort=10.5 velocity=1000.0 -> lower=-4.88692 upper=3.14159 effort=10.5 velocity=3.0; origin xyz=0.00000 -0.01400 0.21100 rpy=0.00000 0.249176479 0.00000 -> xyz=0.00000 -0.01400 0.21100 rpy=0.00000 0.00000 0.00000
- joint Joint_5: limit lower=-3.14159 upper=3.14159 effort=10.5 velocity=1000.0 -> lower=-3.14159 upper=3.14159 effort=10.5 velocity=3.0; origin xyz=0.00000 0.04700 0.03900 rpy=0.00000 0.00000 1.556765769 -> xyz=0.00000 0.04700 0.03900 rpy=0.00000 0.00000 0.00000
- joint Joint_6: axis 0.00000 -1.00000 0.00000 -> 0.00000 1.00000 0.00000; limit lower=-12.5664 upper=12.5664 effort=40.0 velocity=1000.0 -> lower=-12.5664 upper=12.5664 effort=40.0 velocity=3.14; origin xyz=0.00000 0.06080 0.04700 rpy=0.00000 -0.000479370 0.00000 -> xyz=0.00000 0.06080 0.04700 rpy=0.00000 0.00000 0.00000

File: eRob_moveit/src/eRob_ROS2_MoveIt/zeroerr/config/urdfs/eRobo3.ros2_control.xacro (robot description, xacro)
@@ -30,4 +30,7 @@
                     <state_interface name="error_code"/>
                     <state_interface name="mode_display"/>
+                    <state_interface name="following_error_actual"/>
+                    <state_interface name="torque_sensor"/>
+                    <state_interface name="motor_actual_current"/>
                     <ec_module name="zero_err1">
                         <plugin>ethercat_generic_plugins/EcCiA402Drive</plugin>
@@ -52,4 +55,7 @@
                     <state_interface name="error_code"/>
                     <state_interface name="mode_display"/>
+                    <state_interface name="following_error_actual"/>
+                    <state_interface name="torque_sensor"/>
+                    <state_interface name="motor_actual_current"/>
                     <ec_module name="zero_err2">
                         <plugin>ethercat_generic_plugins/EcCiA402Drive</plugin>
@@ -74,4 +80,7 @@
                     <state_interface name="error_code"/>
                     <state_interface name="mode_display"/>
+                    <state_interface name="following_error_actual"/>
+                    <state_interface name="torque_sensor"/>
+                    <state_interface name="motor_actual_current"/>
                     <ec_module name="zero_err3">
                         <plugin>ethercat_generic_plugins/EcCiA402Drive</plugin>
@@ -96,4 +105,7 @@
                     <state_interface name="error_code"/>
                     <state_interface name="mode_display"/>
+                    <state_interface name="following_error_actual"/>
+                    <state_interface name="torque_sensor"/>
+                    <state_interface name="motor_actual_current"/>
                     <ec_module name="zero_err4">
                         <plugin>ethercat_generic_plugins/EcCiA402Drive</plugin>
@@ -118,4 +130,7 @@
                     <state_interface name="error_code"/>
                     <state_interface name="mode_display"/>
+                    <state_interface name="following_error_actual"/>
+                    <state_interface name="torque_sensor"/>
+                    <state_interface name="motor_actual_current"/>
                     <ec_module name="zero_err5">
                         <plugin>ethercat_generic_plugins/EcCiA402Drive</plugin>
@@ -140,4 +155,7 @@
                     <state_interface name="error_code"/>
                     <state_interface name="mode_display"/>
+                    <state_interface name="following_error_actual"/>
+                    <state_interface name="torque_sensor"/>
+                    <state_interface name="motor_actual_current"/>
                     <ec_module name="zero_err6">
                         <plugin>ethercat_generic_plugins/EcCiA402Drive</plugin>
